Commit message: улучшил читаемость файла base.urdf

File: quetzalcoatl_description/urdf/base.urdf.xacro (robot description, xacro)
@@ -7,7 +7,5 @@
 	<link name="base_center">
 		<visual>
-			<origin
-					xyz="0 0 0"
-					rpy="0 0 0" />
+			<origin xyz="0 0 0" rpy="0 0 0" />
 			<geometry>
 				<box size="${body_length} ${body_width} ${body_heigth}" />
@@ -15,7 +13,5 @@
 		</visual>
 		<collision>
-			<origin
-					xyz="0 0 0"
-					rpy="0 0 0" />
+			<origin xyz="0 0 0" rpy="0 0 0" />
 			<geometry>
 				<box size="${body_length} ${body_width} ${body_heigth}" />
@@ -27,14 +23,10 @@
 				height="${body_heigth}"
 				mass="${body_mass}">
-			<origin
-					xyz="0 0 0"
-					rpy="0 0 0" />
+			<origin xyz="0 0 0" rpy="0 0 0" />
 		</xacro:box_inertia>
 	</link>
 	<link name="nose_center">
 		<visual>
-			<origin
-					xyz="0 0 0"
-					rpy="0 0 0" />
+			<origin xyz="0 0 0" rpy="0 0 0" />
 			<geometry>
 				<box size="${nose_length} ${nose_width} ${nose_heigth}" />
@@ -42,7 +34,5 @@
 		</visual>
 		<collision>
-			<origin
-					xyz="0 0 0"
-					rpy="0 0 0" />
+			<origin xyz="0 0 0" rpy="0 0 0" />
 			<geometry>
 				<box size="${nose_length} ${nose_width} ${nose_heigth}" />
@@ -54,7 +44,5 @@
 				height="${nose_heigth}"
 				mass="${nose_mass}">
-			<origin
-					xyz="0 0 0"
-					rpy="0 0 0" />
+			<origin xyz="0 0 0" rpy="0 0 0" />
 		</xacro:box_inertia>
 	</link>
@@ -68,44 +56,26 @@
 	<link name="base_front_axis_link" />
 	<gazebo reference="base_front_axis_link" />
-	<joint
-			name="base_footprint_2_link"
-			type="fixed">
+	<joint name="base_footprint_2_link" type="fixed">
 		<parent link="base_footprint" />
 		<child link="base_link" />
-		<origin
-				xyz="0 0 ${wheel_radius}"
-				rpy="0 0 0" />
+		<origin xyz="0 0 ${wheel_radius}" rpy="0 0 0" />
 	</joint>
-	<joint
-			name="base_link_2_center"
-			type="fixed">
+	<joint name="base_link_2_center" type="fixed">
 		<parent link="base_link" />
 		<child link="base_center" />
-		<origin
-				xyz="${body_length/2-rear_wheel_2_bumper} 0 ${body_heigth/2}"
-				rpy="0 0 0" />
+		<origin xyz="${body_length/2-rear_wheel_2_bumper} 0 ${body_heigth/2}" rpy="0 0 0" />
 	</joint>
-	<joint
-			name="base_link_2_front_axis"
-			type="fixed">
+	<joint name="base_link_2_front_axis" type="fixed">
 		<parent link="base_link" />
 		<child link="base_front_axis_link" />
-		<origin
-				xyz="${wheelbase} 0 0"
-				rpy="0 0 0" />
+		<origin xyz="${wheelbase} 0 0" rpy="0 0 0" />
 	</joint>
-	<joint
-			name="base_front_axis_2_nose_center"
-			type="fixed">
+	<joint name="base_front_axis_2_nose_center" type="fixed">
 		<parent link="base_front_axis_link" />
 		<child link="nose_center" />
-		<origin
-				xyz="${nose_length/2} 0 ${nose_heigth/2}"
-				rpy="0 0 0" />
+		<origin xyz="${nose_length/2} 0 ${nose_heigth/2}" rpy="0 0 0" />
 	</joint>
 	<gazebo>
-		<plugin
-				name="interface_plugin"
-				filename="libackermann_controller_plugin.so">
+		<plugin name="interface_plugin" filename="libackermann_controller_plugin.so">
 			<debug>false</debug>
 			<maxSteerRad>${wheel_mid_turn_limit}</maxSteerRad>

Commit message: расставил основные детали описания по порядку их зависимости друг от друга, добавил `gazebo reference` где этого не хватало

File: quetzalcoatl_description/urdf/base.urdf.xacro (robot description, xacro)
@@ -4,5 +4,21 @@
 	<xacro:include filename="$(find maddrive_urdf_tools)/urdf/macros/wheels.urdf.xacro" />
 	<xacro:include filename="$(find maddrive_urdf_tools)/urdf/macros/inertia.urdf.xacro" />
-	<!-- Large box =) -->
+	<!-- BASE FOOTPRINT-->
+	<link name="base_footprint" />
+	<gazebo reference="base_footprint" />
+	<joint name="base_footprint_2_base_link" type="fixed">
+		<parent link="base_footprint" />
+		<child link="base_link" />
+		<origin xyz="0 0 ${wheel_radius}" rpy="0 0 0" />
+	</joint>
+	<!-- BASE LINK-->
+	<link name="base_link" />
+	<gazebo reference="base_link" />
+	<joint name="base_link_2_base_center" type="fixed">
+		<parent link="base_link" />
+		<child link="base_center" />
+		<origin xyz="${body_length/2-rear_wheel_2_bumper} 0 ${body_heigth/2}" rpy="0 0 0" />
+	</joint>
+	<!-- BASE CENTER -->
 	<link name="base_center">
 		<visual>
@@ -26,4 +42,19 @@
 		</xacro:box_inertia>
 	</link>
+	<gazebo reference="base_center" />
+	<joint name="base_link_2_base_front_axis_link" type="fixed">
+		<parent link="base_link" />
+		<child link="base_front_axis_link" />
+		<origin xyz="${wheelbase} 0 0" rpy="0 0 0" />
+	</joint>
+	<!-- BASE FRONT AXIS LINK-->
+	<link name="base_front_axis_link" />
+	<gazebo reference="base_front_axis_link" />
+	<joint name="base_front_axis_link_2_nose_center" type="fixed">
+		<parent link="base_front_axis_link" />
+		<child link="nose_center" />
+		<origin xyz="${nose_length/2} 0 ${nose_heigth/2}" rpy="0 0 0" />
+	</joint>
+	<!-- NOSE_CENTER-->
 	<link name="nose_center">
 		<visual>
@@ -47,34 +78,28 @@
 		</xacro:box_inertia>
 	</link>
-	<!-- BASE FOOTPRINT-->
-	<link name="base_footprint" />
-	<gazebo reference="base_footprint" />
-	<!-- BASE LINK-->
-	<link name="base_link" />
-	<gazebo reference="base_link" />
-	<!-- BASE FRONT AXIS LINK-->
-	<link name="base_front_axis_link" />
-	<gazebo reference="base_front_axis_link" />
-	<joint name="base_footprint_2_link" type="fixed">
-		<parent link="base_footprint" />
-		<child link="base_link" />
-		<origin xyz="0 0 ${wheel_radius}" rpy="0 0 0" />
-	</joint>
-	<joint name="base_link_2_center" type="fixed">
-		<parent link="base_link" />
-		<child link="base_center" />
-		<origin xyz="${body_length/2-rear_wheel_2_bumper} 0 ${body_heigth/2}" rpy="0 0 0" />
-	</joint>
-	<joint name="base_link_2_front_axis" type="fixed">
-		<parent link="base_link" />
-		<child link="base_front_axis_link" />
-		<origin xyz="${wheelbase} 0 0" rpy="0 0 0" />
-	</joint>
-	<joint name="base_front_axis_2_nose_center" type="fixed">
-		<parent link="base_front_axis_link" />
-		<child link="nose_center" />
-		<origin xyz="${nose_length/2} 0 ${nose_heigth/2}" rpy="0 0 0" />
-	</joint>
+	<gazebo reference="nose_center" />
+	<xacro:steer_wheel
+			name="front_right_wheel"
+			base_name="base_link"
+			xyz="${wheelbase} -${track_width/2} 0"
+			steer_limit="${wheel_mid_turn_limit}" />
+	<xacro:steer_wheel
+			name="front_left_wheel"
+			base_name="base_link"
+			xyz="${wheelbase} ${track_width/2} 0"
+			steer_limit="${wheel_mid_turn_limit}" />
+	<xacro:speed_wheel
+			name="rear_right_wheel"
+			base_name="base_link"
+			xyz="0 -${track_width/2} 0" />
+	<xacro:speed_wheel
+			name="rear_left_wheel"
+			base_name="base_link"
+			xyz="0 ${track_width/2} 0" />
 	<gazebo>
+		<!-- <plugin name="gazebo_ros_control" filename="libgazebo_ros_control.so">
+			<robotNamespace>/</robotNamespace>
+			<robotSimType>gazebo_ros_control/DefaultRobotHWSim</robotSimType>
+		</plugin> -->
 		<plugin name="interface_plugin" filename="libackermann_controller_plugin.so">
 			<debug>false</debug>
@@ -117,21 +142,3 @@
 		</plugin>
 	</gazebo>
-	<xacro:steer_wheel
-			name="front_right_wheel"
-			base_name="base_link"
-			xyz="${wheelbase} -${track_width/2} 0"
-			steer_limit="${wheel_mid_turn_limit}" />
-	<xacro:steer_wheel
-			name="front_left_wheel"
-			base_name="base_link"
-			xyz="${wheelbase} ${track_width/2} 0"
-			steer_limit="${wheel_mid_turn_limit}" />
-	<xacro:speed_wheel
-			name="rear_right_wheel"
-			base_name="base_link"
-			xyz="0 -${track_width/2} 0" />
-	<xacro:speed_wheel
-			name="rear_left_wheel"
-			base_name="base_link"
-			xyz="0 ${track_width/2} 0" />
 </robot>

Commit message: переименовал основной лаунч симуляции на общий манер, добавил модель настоящей газели, настроил визуал модели, немного поднастрил отображение в rviz

File: quetzalcoatl_description/urdf/base.urdf.xacro (robot description, xacro)
@@ -13,5 +13,12 @@
 	</joint>
 	<!-- BASE LINK-->
-	<link name="base_link" />
+	<link name="base_link">
+		<visual>
+			<origin xyz="0 0 0" rpy="0 0 0" />
+			<geometry>
+				<mesh filename="package://quetzalcoatl_description/meshes/gazelle-next.dae" />
+			</geometry>
+		</visual>
+	</link>
 	<gazebo reference="base_link" />
 	<joint name="base_link_2_base_center" type="fixed">
@@ -22,10 +29,4 @@
 	<!-- BASE CENTER -->
 	<link name="base_center">
-		<visual>
-			<origin xyz="0 0 0" rpy="0 0 0" />
-			<geometry>
-				<box size="${body_length} ${body_width} ${body_heigth}" />
-			</geometry>
-		</visual>
 		<collision>
 			<origin xyz="0 0 0" rpy="0 0 0" />
@@ -58,10 +59,4 @@
 	<!-- NOSE_CENTER-->
 	<link name="nose_center">
-		<visual>
-			<origin xyz="0 0 0" rpy="0 0 0" />
-			<geometry>
-				<box size="${nose_length} ${nose_width} ${nose_heigth}" />
-			</geometry>
-		</visual>
 		<collision>
 			<origin xyz="0 0 0" rpy="0 0 0" />

File: quetzalcoatl_description/urdf/robocross_22.urdf.xacro (robot description, xacro)
@@ -1,5 +1,5 @@
 <?xml version="1.0"?>
 <robot
-		name="gazel"
+		name="gazelle"
 		xmlns:xacro="http://www.ros.org/wiki/xacro">
 	<xacro:include filename="$(find quetzalcoatl_description)/urdf/base.urdf.xacro" />

Commit message: описание переработано так, чтобы был порядок "сочлинение - деталь", добавлены макросы-маркеты отсутствия моделей

File: quetzalcoatl_description/urdf/base.urdf.xacro (robot description, xacro)
@@ -4,7 +4,13 @@
 	<xacro:include filename="$(find maddrive_urdf_tools)/urdf/macros/wheels.urdf.xacro" />
 	<xacro:include filename="$(find maddrive_urdf_tools)/urdf/macros/inertia.urdf.xacro" />
+	<xacro:include filename="$(find maddrive_urdf_tools)/urdf/macros/common.urdf.xacro" />
 	<!-- BASE FOOTPRINT-->
-	<link name="base_footprint" />
+	<link name="base_footprint">
+		<xacro:null_visual/>
+		<xacro:null_collision/>
+		<xacro:null_inertia/>
+	</link>
 	<gazebo reference="base_footprint" />
+	<!-- BASE LINK-->
 	<joint name="base_footprint_2_base_link" type="fixed">
 		<parent link="base_footprint" />
@@ -12,5 +18,4 @@
 		<origin xyz="0 0 ${wheel_radius}" rpy="0 0 0" />
 	</joint>
-	<!-- BASE LINK-->
 	<link name="base_link">
 		<visual>
@@ -20,6 +25,9 @@
 			</geometry>
 		</visual>
+		<xacro:null_collision/>
+		<xacro:null_inertia/>
 	</link>
 	<gazebo reference="base_link" />
+	<!-- BASE CENTER -->
 	<joint name="base_link_2_base_center" type="fixed">
 		<parent link="base_link" />
@@ -27,6 +35,6 @@
 		<origin xyz="${body_length/2-rear_wheel_2_bumper} 0 ${body_heigth/2}" rpy="0 0 0" />
 	</joint>
-	<!-- BASE CENTER -->
 	<link name="base_center">
+		<xacro:null_visual/>
 		<collision>
 			<origin xyz="0 0 0" rpy="0 0 0" />
@@ -44,4 +52,5 @@
 	</link>
 	<gazebo reference="base_center" />
+	<!-- BASE FRONT AXIS LINK-->
 	<joint name="base_link_2_base_front_axis_link" type="fixed">
 		<parent link="base_link" />
@@ -49,7 +58,11 @@
 		<origin xyz="${wheelbase} 0 0" rpy="0 0 0" />
 	</joint>
-	<!-- BASE FRONT AXIS LINK-->
-	<link name="base_front_axis_link" />
+	<link name="base_front_axis_link">
+		<xacro:null_visual/>
+		<xacro:null_collision/>
+		<xacro:null_inertia/>
+	</link>
 	<gazebo reference="base_front_axis_link" />
+	<!-- NOSE_CENTER-->
 	<joint name="base_front_axis_link_2_nose_center" type="fixed">
 		<parent link="base_front_axis_link" />
@@ -57,6 +70,6 @@
 		<origin xyz="${nose_length/2} 0 ${nose_heigth/2}" rpy="0 0 0" />
 	</joint>
-	<!-- NOSE_CENTER-->
 	<link name="nose_center">
+		<xacro:null_visual/>
 		<collision>
 			<origin xyz="0 0 0" rpy="0 0 0" />
@@ -74,4 +87,5 @@
 	</link>
 	<gazebo reference="nose_center" />
+	<!-- WHEELS-->
 	<xacro:steer_wheel
 			prefix="front_right"
